Commit message: add test environment + BUG algorithm

File: urdf/my_robot_tutorial.urdf (robot description, URDF)
Before this commit: robot my_robot, 7 links, 6 joints
Joints:
- joint hokuyo_joint: origin xyz=0.70 0 0.075 rpy=0 0 0 -> xyz=0 0 0.25 rpy=0 0 0

Commit message: add some

File: urdf/my_robot_tutorial.urdf (robot description, URDF)
Before this commit: robot my_robot, 7 links, 6 joints
Links:
- link left_wheel: geometry collision cylinder length=0.001 radius=0.2; visual cylinder length=0.001 radius=0.2
- link right_wheel: geometry collision cylinder length=0.001 radius=0.2; visual cylinder length=0.001 radius=0.2
